File: Dell 5-6pin 2.0mm Front Panel Header Adapter/Kicad Schematic/Dell 6pin 2.0mm Front Panel Header Adapter.sch (KiCad schematic (older format))
At the start: 2 parts, among them J1 Dell Connector, J2 2.54mm Panel Header

Commit message: redesign PCB to fit (more) Micro ATX cases
The original PCB hung off the side of the motherboard.
If the motherboard is mounted very close to the power
supply, the PCB won't physically fit.

One example of a case with this issue is the Rosewill
LINE-M.

The redesigned PCB should (hopefully) not hang off
edge of the motherboard at all.  I don't believe it
will physically obstruct any other connector, but I
haven't had it fabbed yet, so we'll see.
Parts:
- J1, J2: symbol Connector_Generic:Conn_02x03_Odd_Even -> Dell-6pin-2.0mm-Front-Panel-Header-Adapter-rescue:Conn_02x03_Odd_Even-Connector_Generic
Changed lines of the file:
@@
 EESchema Schematic File Version 4
-LIBS:Dell 6pin 2.0mm Front Panel Header Adapter-cache
-EELAYER 29 0
+EELAYER 30 0
 EELAYER END
 $Descr A4 11693 8268
@@
 $EndDescr
 $Comp
-L Connector_Generic:Conn_02x03_Odd_Even J2
+L Dell-6pin-2.0mm-Front-Panel-Header-Adapter-rescue:Conn_02x03_Odd_Even-Connector_Generic J2
 U 1 1 5D44D227
 P 4800 3700
@@
 $EndComp
 $Comp
-L Connector_Generic:Conn_02x03_Odd_Even J1
+L Dell-6pin-2.0mm-Front-Panel-Header-Adapter-rescue:Conn_02x03_Odd_Even-Connector_Generic J1
 U 1 1 5D44F1CB
 P 4800 3150
